File: UglyFace_01.kicad_sch (KiCad schematic)
At the start: 31 parts, among them J1 9V, J2 9V GND, J3 IN/LED/LG/OUT, J4 IN GND, J6 OUT GND, U1 LM386, U2 TLC555, U3 Vactrol

Commit message: Ugly Face 1 v1.2: THR toggle, CMOS protection, 3362P GLITCH trimmer, new control layout
As ordered from JLCPCB (October 2026 batch).

Co-Authored-By: Claude Opus 5.5 <noreply@anthropic.com>
Parts:
- added R10, R8: 1k, Resistor_SMD:R_0805_2012Metric_Pad1.20x1.40mm_HandSolder, symbol Device:R
- added R7: 2k2, Resistor_SMD:R_0805_2012Metric_Pad1.20x1.40mm_HandSolder, symbol Device:R
- added R9: 22k, Resistor_SMD:R_0805_2012Metric_Pad1.20x1.40mm_HandSolder, symbol Device:R
- added SW1: THR, UglyFace:SW_Taiway_100_SPDT_PC, symbol Switch:SW_SPDT
- C5: value 100u -> 22u; footprint Capacitor_SMD:CP_Elec_6.3x7.7 -> Capacitor_SMD:C_1206_3216Metric_Pad1.33x1.80mm_HandSolder; symbol Device:C_Polarized -> Device:C; FT Rotation Offset 180 -> (none); LCSC C970685 -> C12891
- D2, RV1, RV3, RV4, U3: now left out of the parts list
- RV2: value B10k -> 10k; footprint UglyFace:Potentiometer_Alpha_16mm_Vertical -> UglyFace:Potentiometer_Bourns_3362P_Vertical; symbol Device:R_Potentiometer -> Device:R_Potentiometer_Trim; Label THR -> GLITCH; now left out of the parts list
Connections:
- net +9V: now also R7.1
- net DISCH: now also R10.1; no longer C7.1
- net GND: now also R8.2
- net RESET: now also R9.2; no longer C4.2, RV2.2
- new net: R7.2, SW1.3 (C)
- new net: R8.1, SW1.1 (A)
- new net: C7.1, R10.2
- new net: C4.2, R9.1, RV2.2, SW1.2 (B)
Other:
- note added: "R9: 22k into RESET limits current from the gate swing (TLC555 pin 4 was being driven to -0.75 V)."
- note added: "THRESHOLD = SW1 toggle: GATED (R8) / GLITCH (centre, RV2 trim) / ON (R7)"
- note removed: "THRESHOLD"
