File: UglyFace_01.kicad_pcb (KiCad board)
At the start: 2 copper layers, 50.5 x 32.7 mm, 32 parts, among them J1 9V, J2 9V GND, J3 IN/LED/LG/OUT, J4 IN GND, J6 OUT GND, U1 LM386, U2 TLC555, U3 Vactrol

Commit message: Ugly Face 1 v1.2: THR toggle, CMOS protection, 3362P GLITCH trimmer, new control layout
As ordered from JLCPCB (October 2026 batch).

Co-Authored-By: Claude Opus 5.5 <noreply@anthropic.com>
Parts:
- added R10: 1k, Resistor_SMD:R_0805_2012Metric_Pad1.20x1.40mm_HandSolder, F.Cu at (168.3, 109.0)
- added R7: 2k2, Resistor_SMD:R_0805_2012Metric_Pad1.20x1.40mm_HandSolder, F.Cu at (146.0, 107.0)
- added R8: 1k, Resistor_SMD:R_0805_2012Metric_Pad1.20x1.40mm_HandSolder, F.Cu at (154.0, 107.0)
- added R9: 22k, Resistor_SMD:R_0805_2012Metric_Pad1.20x1.40mm_HandSolder, F.Cu at (161.5, 109.5)
- added SW1: THR, UglyFace:SW_Taiway_100_SPDT_PC, B.Cu at (134.1, 102.9)
- C5: value 100u -> 22u; footprint Capacitor_SMD:CP_Elec_6.3x7.7 -> Capacitor_SMD:C_1206_3216Metric_Pad1.33x1.80mm_HandSolder
- RV2: value B10k -> 10k; footprint UglyFace:Potentiometer_Alpha_16mm_Vertical -> UglyFace:Potentiometer_Bourns_3362P_Vertical
- moved RV1 38.2 mm to (162.6, 118.9)
- moved RV3 38.2 mm to (134.1, 93.5)
- moved RV4 38.2 mm to (162.6, 93.5)
- moved D1 14.0 mm to (135.3, 111.0)
- moved RV2 5.34 mm to (163.2, 98.8), turned to 90 degrees
- moved C10 3.50 mm to (155.0, 110.1)
- moved U2 2.26 mm to (163.7, 105.2)
- moved U1 2.00 mm to (147.8, 110.8)
- moved C6 1.50 mm to (158.5, 108.5)
- moved C1 1.25 mm to (125.4, 100.3)
- moved C5 1.00 mm to (130.0, 106.5)
- moved C2 0.25 mm to (140.8, 116.4)
Connections:
- C4 pad 2: /RESET -> Net-(SW1-B)
- C7 pad 1: /DISCH -> Net-(C7-Pad1)
- RV2 pad 2: /RESET -> Net-(SW1-B)
Routing:
- net Net-(SW1-B): track 0.00 -> 55.8 mm, vias 0 -> 2
- net Net-(C7-Pad1): track 0.00 -> 54.7 mm
- net Net-(R2-Pad1): track 3.82 -> 47.2 mm, vias 0 -> 1
- net Net-(C7-Pad2): track 6.39 -> 44.6 mm, vias 0 -> 1
- net Net-(SW1-A): track 0.00 -> 23.4 mm
- net /DISCH: track 64.8 -> 46.2 mm, vias 0 -> 2
- net /RESET: track 20.7 -> 2.95 mm, vias 2 -> 0
- net Net-(C5-Pad2): track 16.2 -> 33.7 mm, vias 1 -> 0
- net /AMP_OUT: track 37.2 -> 53.7 mm, vias 2 -> 0
- net Net-(SW1-C): track 0.00 -> 13.5 mm
- net +9V: track 100.8 -> 111.2 mm, vias 3 -> 0
- net Net-(R4-Pad2): track 15.1 -> 5.81 mm
- net /VACT_LED: track 26.2 -> 35.2 mm
- net /TIMING: track 49.9 -> 41.6 mm
- net /OUT: track 20.0 -> 28.4 mm
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Other:
- board text added: "SUPER-FREQ"
- board text added: "UGLY FACE v1.2"

Commit message: Ugly Face 1: v1.2 test sheet and 555 debug notes, v1.2 KiCad archive, Envelope A breadboard, toggle slot footprint, vactrol LED resistor note
Co-Authored-By: Claude Opus 5.5 <noreply@anthropic.com>
Routing:
- net +9V: track 111.2 -> 97.2 mm, vias 0 -> 5
- net Net-(SW1-B): track 55.8 -> 43.7 mm, vias 2 -> 3
- net /VACT_LED: track 35.2 -> 25.2 mm
- net /OSC_SQ: track 34.6 -> 43.4 mm
- net /OUT: track 28.4 -> 33.6 mm
- net /TIMING: track 41.6 -> 46.7 mm
- net Net-(R2-Pad1): track 47.2 -> 42.7 mm
- net /DISCH: track 46.2 -> 41.9 mm
- net Net-(C7-Pad1): track 54.7 -> 50.9 mm, vias 0 -> 2
- net GND: track 171.5 -> 167.8 mm, vias 1 -> 4
- net Net-(R5-Pad1): track 6.19 -> 9.50 mm
- net /IN: track 10.7 -> 12.0 mm, vias 0 -> 1
- net /LED_K: track 25.2 -> 26.5 mm
- net Net-(C5-Pad2): track 33.7 -> 32.5 mm, vias 0 -> 1
- net Net-(U1-BYPASS): track 5.54 -> 6.47 mm, vias 0 -> 2
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